Commit message: world added

File: description/robot.urdf.xacro (robot description, xacro)
@@ -2,3 +2,4 @@
 <robot xmlns:xacro="http://www.ros.org/wiki/xacro"  name="robot">
     <xacro:include filename="robot_core.xacro" />
+    <xacro:include filename="gazebo_control.xacro" />
 </robot>

File: description/robot_core.xacro (robot description, xacro)
@@ -41,4 +41,7 @@
         </xacro:inertial_box>
     </link>
+    <gazebo reference="chassis">
+        <material>Gazebo/White</material>
+    </gazebo>
     <!-- Left Wheel link -->
     <joint name="left_wheel_joint" type="continuous">
@@ -64,4 +67,7 @@
         </xacro:inertial_cylinder>
     </link>
+    <gazebo reference="left_wheel">
+        <material>Gazebo/Blue</material>
+    </gazebo>
      <!-- Rigth Wheel link -->
     <joint name="rigth_wheel_joint" type="continuous">
@@ -87,4 +93,7 @@
         </xacro:inertial_cylinder>
     </link>
+    <gazebo reference="right_wheel">
+        <material>Gazebo/Blue</material>
+    </gazebo>
      <!-- Caster Wheel link -->
     <joint name="caster_wheel_joint" type="fixed">
@@ -109,3 +118,8 @@
         </xacro:inertial_sphere>
     </link>
+    <gazebo reference="caster_wheel">
+        <material>Gazebo/Black</material>
+        <mu1 value="0.001"/>
+        <mu2 value="0.001"/>
+    </gazebo>
 </robot>

Commit message: camera and lidar

File: description/robot.urdf.xacro (robot description, xacro)
@@ -3,3 +3,5 @@
     <xacro:include filename="robot_core.xacro" />
     <xacro:include filename="gazebo_control.xacro" />
+    <xacro:include filename="lidar.xacro" />
+    <xacro:include filename="camera.xacro" />
 </robot>

File: description/robot_core.xacro (robot description, xacro)
@@ -14,14 +14,17 @@
         <color rgba="0 0 0 1" />
     </material>
+    <material name="red">
+        <color rgba="1 0 0 1"/>
+    </material>
     <!-- Base link -->
     <link name="base_link">
     </link>
-    <!-- Chasis link -->
-    <joint name="chasis_joint" type="fixed">
+    <!-- chassis link -->
+    <joint name="chassis_joint" type="fixed">
         <parent link="base_link" />
-        <child link="chasis" />
+        <child link="chassis" />
         <origin xyz="-0.1 0 0" />
     </joint>
-    <link name="chasis">
+    <link name="chassis">
         <visual>
             <origin xyz="0.15 0 0.075" />
@@ -93,10 +96,10 @@
         </xacro:inertial_cylinder>
     </link>
-    <gazebo reference="right_wheel">
+    <gazebo reference="rigth_wheel">
         <material>Gazebo/Blue</material>
     </gazebo>
      <!-- Caster Wheel link -->
     <joint name="caster_wheel_joint" type="fixed">
-        <parent link="chasis" />
+        <parent link="chassis" />
         <child link="caster_wheel" />
         <origin xyz="0.24 0 0" />

Commit message: new update

File: description/robot.urdf.xacro (robot description, xacro)
@@ -2,6 +2,8 @@
 <robot xmlns:xacro="http://www.ros.org/wiki/xacro"  name="robot">
     <xacro:include filename="robot_core.xacro" />
-    <xacro:include filename="gazebo_control.xacro" />
+    <!-- <xacro:include filename="gazebo_control.xacro" /> -->
+    <xacro:include filename="ros2_control.xacro" />
     <xacro:include filename="lidar.xacro" />
     <xacro:include filename="camera.xacro" />
+    <!-- <xacro:include filename="depth_camera.xacro" /> -->
 </robot>

File: description/robot_core.xacro (robot description, xacro)
@@ -63,5 +63,5 @@
         <collision>
             <geometry>
-                <cylinder radius="0.05" length="0.04"/>
+                <sphere radius="0.05" />
             </geometry>
         </collision>
@@ -73,12 +73,12 @@
         <material>Gazebo/Blue</material>
     </gazebo>
-     <!-- Rigth Wheel link -->
-    <joint name="rigth_wheel_joint" type="continuous">
+     <!-- Right Wheel link -->
+    <joint name="right_wheel_joint" type="continuous">
         <parent link="base_link" />
-        <child link="rigth_wheel" />
+        <child link="right_wheel" />
         <origin xyz="0 -0.175 0" rpy="${pi/2} 0 0" />
         <axis xyz="0 0 -1" />
     </joint>
-    <link name="rigth_wheel">
+    <link name="right_wheel">
         <visual>
             <geometry>
@@ -89,5 +89,5 @@
         <collision>
             <geometry>
-                <cylinder radius="0.05" length="0.04"/>
+                <sphere radius="0.05" />
             </geometry>
         </collision>
@@ -96,5 +96,5 @@
         </xacro:inertial_cylinder>
     </link>
-    <gazebo reference="rigth_wheel">
+    <gazebo reference="right_wheel">
         <material>Gazebo/Blue</material>
     </gazebo>
